File: IFS09-ControlBoard/IFS09-ControlBoard.kicad_pcb (KiCad board)
At the start: 2 copper layers, 65 x 60 mm, 74 parts, among them J1 1-776087-1, J2 Conn_01x04_Pin, J3 Conn_01x04_Pin, J4 Conn_01x05_Pin, SW1 SW_Push, U1 TSR_1-2450, U2 LM2936-3.3_TO92, U3 TCAN330, U4 STM32H7A3IGTxQ, U5 TCAN330, Y1 XUX53

Commit message: Add files via upload
Parts:
- moved R5 5.62 mm to (205.0, 56.3), turned to 90 degrees
- moved C4 0.77 mm to (187.4, 57.9)
Connections:
- net /CAN1_H renamed /CAN1_P
- net /CAN1_L renamed /CAN1_N
- net /CAN2_H renamed /CAN2_P
- net /CAN2_L renamed /CAN2_N
Routing:
- net /NRST: track 43.0 -> 48.2 mm
- net /CAN1_N: track 14.4 -> 18.8 mm
- net /CAN2_N: track 11.3 -> 15.4 mm
- net GND: track 44.9 -> 47.9 mm, vias 37 -> 38
- net /CAN1_P: track 16.6 -> 18.9 mm
- net /CAN2_P: track 13.6 -> 15.3 mm
Other:
- board size 65 x 60 mm -> 65 x 61.6 mm
