File: IFS09-ControlBoard/IFS09-ControlBoard.kicad_sch (KiCad schematic)
At the start: 74 parts, among them J1 1-776087-1, J2 Conn_01x04_Pin, J3 Conn_01x04_Pin, J4 Conn_01x05_Pin, SW1 SW_Push, U1 TSR_1-2450, U2 LM2936-3.3_TO92, U3 TCAN330, U4 STM32H7A3IGTxQ, U5 TCAN330, Y1 XUX53

Commit message: Add files via upload
Connections:
- net CAN1_H renamed CAN1_P
- net CAN1_L renamed CAN1_N
- net CAN2_H renamed CAN2_P
- net CAN2_L renamed CAN2_N
Changed lines of the file:
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@@
 		)
 	)
-	(label "CAN1_L"
+	(label "CAN1_N"
 		(at 88.9 262.89 0)
 		(effects
@@
 		)
 	)
-	(label "CAN1_H"
+	(label "CAN1_P"
 		(at 88.9 254 0)
 		(effects
@@
 		)
 	)
-	(label "CAN1_L"
+	(label "CAN1_N"
 		(at 44.45 58.42 180)
 		(effects
@@
 		)
 	)
-	(label "CAN2_L"
+	(label "CAN2_N"
 		(at 44.45 63.5 180)
 		(effects
@@
 		)
 	)
-	(label "CAN2_H"
+	(label "CAN2_P"
 		(at 44.45 66.04 180)
 		(effects
@@
 		)
 	)
-	(label "CAN1_H"
+	(label "CAN1_P"
 		(at 44.45 60.96 180)
 		(effects
@@
 		)
 	)
-	(label "CAN2_H"
+	(label "CAN2_P"
 		(at 152.4 252.73 0)
 		(effects
@@
 		)
 	)
-	(label "CAN2_L"
+	(label "CAN2_N"
 		(at 152.4 264.16 0)
 		(effects
